Commit message: lalala

File: duck_testing/pybullet_ur5_robotiq/boxes/box_large.urdf (robot description, URDF)
Before this commit: robot large_box, 1 links, 0 joints
Links:
- link base: geometry collision box size=0.05 0.11 0.05; visual box size=0.05 0.11 0.05

File: duck_testing/pybullet_ur5_robotiq/boxes/box_medium.urdf (robot description, URDF)
Before this commit: robot medium_box, 1 links, 0 joints
Links:
- link base: geometry collision box size=0.05 0.08 0.05; visual box size=0.05 0.08 0.05
