Commit message: add boxes, fixed gravity physics, arm points the right way always

File: main/UArm_robot/boxes/box_large.urdf (robot description, URDF)
Before this commit: robot large_box, 1 links, 0 joints
Links:
- link base: geometry collision box size=0.025 0.06 0.025; visual box size=0.05 0.04 0.025

File: main/UArm_robot/boxes/box_medium.urdf (robot description, URDF)
Before this commit: robot medium_box, 1 links, 0 joints
Links:
- link base: geometry collision box size=0.025 0.04 0.025; visual box size=0.04 0.04 0.025

File: main/UArm_robot/boxes/box_small.urdf (robot description, URDF)
Before this commit: robot small_box, 1 links, 0 joints
Links:
- link base: geometry collision box size=0.025 0.025 0.025; visual box size=0.025 0.04 0.025

File: main/UArm_robot/urdf/UArm.urdf (robot description, URDF)
Before this commit: robot UArm, 7 links, 6 joints
Links:
- added link link6, mass 0.1; visual mesh filename=../meshes/Link5.stl scale=0.001 0.001 0.001
Joints:
- added joint joint5: type revolute, parent link5, child link6, origin xyz=0 -0.035 -0.045 rpy=0 0 0, axis 0 0 1, limit lower=-6.28 upper=6.28 effort=10 velocity=1
- joint camera_joint: origin xyz=0.02 0 0.05 rpy=0 1.57 -1.57 -> xyz=0.02 -0.035 0.00 rpy=0 1.57 -1.57; parent tool -> link5
- joint tool_joint: origin xyz=0.0 -0.035 -0.06 rpy=0 0 0 -> xyz=0.0 -0.0 -0.01 rpy=0 0 0; parent link5 -> link6
